Commit message: Isaac Sim 6 as the robot: physical billets and a simulated magnet
sim.launch.py hw:=isaac swaps FANUC's mock hardware for Isaac Sim through
topic_based_ros2_control; MoveIt, MTC and pick_drop.cpp are unchanged.

- urdf: hw:=mock|isaac|real (use_mock still works); Isaac ros2_control
  commands position + velocity
- isaac/billet_cell.py: imports the URDF, builds the cell from
  pick_drop.yaml (table mesh, pallets, steel billets), ROS 2 joint/clock
  graph, magnet as a fixed joint with a capture range, contact and
  billet-drift logging, --settle-test
- magnet_bridge: planning-scene attach/detach -> /magnet
- isaac_controllers.yaml: standard JTC, tight goal tolerance
- README section 7: how to run, what the logs mean, lessons learned

Verified headless: 5/5 billets placed within 1 mm of their drop slots;
hw:=mock still 5/5.

Co-Authored-By: Claude Opus 5.5 <noreply@anthropic.com>

File: urdf/crx10ia_l_schmalz.urdf.xacro (robot description, xacro)
@@ -23,11 +23,21 @@
   <xacro:arg name="robot_xyz" default="-0.65 0 0.959"/>
   <xacro:arg name="robot_rpy" default="0 0 0"/>
+  <!-- Hardware: mock | isaac | real. Empty = follow use_mock (official driver argument). -->
+  <xacro:arg name="hw" default=""/>
+  <xacro:property name="hw" value="$(arg hw)"/>
+  <xacro:if value="${hw == ''}">
+    <xacro:if value="$(arg use_mock)"><xacro:property name="hw" value="mock"/></xacro:if>
+    <xacro:unless value="$(arg use_mock)"><xacro:property name="hw" value="real"/></xacro:unless>
+  </xacro:if>
   <xacro:include filename="$(find fanuc_crx_description)/urdf/crx10ia_l_urdf_macro.xacro"/>
-  <xacro:if value="$(arg use_mock)">
+  <xacro:if value="${hw == 'mock'}">
     <xacro:include filename="$(find fanuc_hardware_interface)/config/crx_mock_ros2_control_macro.xacro"/>
   </xacro:if>
-  <xacro:unless value="$(arg use_mock)">
+  <xacro:if value="${hw == 'isaac'}">
+    <xacro:include filename="$(find fanuc_pick_drop)/urdf/crx_isaac_ros2_control.xacro"/>
+  </xacro:if>
+  <xacro:if value="${hw == 'real'}">
     <xacro:include filename="$(find fanuc_hardware_interface)/config/crx_physical_ros2_control_macro.xacro"/>
-  </xacro:unless>
+  </xacro:if>
   <xacro:include filename="$(find moveit_resources_fanuc_moveit_config)/config/schmalz_eoat.urdf.xacro"/>
   <link name="world"/>
